Commit message: latest focused on manual controller only

File: solar_robot_pybullet.urdf (robot description, URDF)
Before this commit: robot solar_cleaning_robot_v2, 24 links, 23 joints
Links:
- removed link bridge_compartment
- removed link bridge_foot_left
- removed link bridge_foot_right
- removed link bridge_segment_1
- removed link bridge_segment_2
- removed link brush_housing
- removed link camera_link
- removed link caster_front_left
- removed link caster_front_right
- removed link imu_link
- removed link lidar_link
- removed link main_suction_pad
- removed link rotating_brush
- removed link squeegee
- removed link suction_chamber
- removed link top_cover
- removed link water_spray_left
- removed link water_spray_right
- removed link wheel_front_left
- removed link wheel_front_right
- removed link wheel_rear_left
- removed link wheel_rear_right
- added link brush, mass 0.14; collision cylinder length=0.32 radius=0.038; visual cylinder length=0.32 radius=0.038
- added link camera; visual box size=0.05 0.025 0.025
- added link front_bridge_base; collision box size=0.10 0.22 0.038; visual box size=0.10 0.22 0.038
- added link front_bridge_seg1, mass 0.11; collision box size=0.15 0.14 0.024; visual box size=0.15 0.14 0.024
- added link front_bridge_seg2, mass 0.09; collision box size=0.15 0.12 0.020; visual box size=0.15 0.12 0.020
- added link front_pad_left, mass 0.015; collision cylinder length=0.007 radius=0.026; visual cylinder length=0.007 radius=0.026
- added link front_pad_right, mass 0.015; collision cylinder length=0.007 radius=0.026; visual cylinder length=0.007 radius=0.026
- added link front_suction_left, mass 0.03; visual cylinder length=0.028 radius=0.007
- added link front_suction_right, mass 0.03; visual cylinder length=0.028 radius=0.007
- added link lidar; visual cylinder length=0.04 radius=0.038
- added link lift_column, mass 0.05; visual box size=0.03 0.03 0.06
- added link rear_bridge_base; collision box size=0.10 0.22 0.038; visual box size=0.10 0.22 0.038
- added link rear_bridge_seg1, mass 0.11; collision box size=0.15 0.14 0.024; visual box size=0.15 0.14 0.024
- added link rear_bridge_seg2, mass 0.09; collision box size=0.15 0.12 0.020; visual box size=0.15 0.12 0.020
- added link rear_pad_left, mass 0.015; collision cylinder length=0.007 radius=0.026; visual cylinder length=0.007 radius=0.026
- added link rear_pad_right, mass 0.015; collision cylinder length=0.007 radius=0.026; visual cylinder length=0.007 radius=0.026
- added link rear_suction_left, mass 0.03; visual cylinder length=0.028 radius=0.007
- added link rear_suction_right, mass 0.03; visual cylinder length=0.028 radius=0.007
- added link wheel_fl, mass 0.20; collision cylinder length=0.022 radius=0.035; visual cylinder length=0.022 radius=0.035
- added link wheel_fr, mass 0.20; collision cylinder length=0.022 radius=0.035; visual cylinder length=0.022 radius=0.035
- added link wheel_rl, mass 0.20; collision cylinder length=0.022 radius=0.035; visual cylinder length=0.022 radius=0.035
- added link wheel_rr, mass 0.20; collision cylinder length=0.022 radius=0.035; visual cylinder length=0.022 radius=0.035
- link base_link: mass 0.01 -> None; geometry 
- link main_body: mass 3.5 -> 3.2; geometry collision box size=0.45 0.35 0.12; visual box size=0.45 0.35 0.12
Joints:
- removed joint base_to_main_body
- removed joint body_to_bridge_compartment
- removed joint body_to_brush_housing
- removed joint body_to_camera
- removed joint body_to_caster_front_left
- removed joint body_to_caster_front_right
- removed joint body_to_cover
- removed joint body_to_imu
- removed joint body_to_lidar
- removed joint body_to_suction
- removed joint body_to_wheel_front_left
- removed joint body_to_wheel_front_right
- removed joint body_to_wheel_rear_left
- removed joint body_to_wheel_rear_right
- removed joint bridge_deploy_joint_1
- removed joint bridge_deploy_joint_2
- removed joint bridge_to_foot_left
- removed joint bridge_to_foot_right
- removed joint brush_rotation_joint
- removed joint brush_to_squeegee
- removed joint housing_to_spray_left
- removed joint housing_to_spray_right
- removed joint suction_to_chamber
- added joint body_lift_joint: type prismatic, parent base_link, child lift_column, origin xyz=0 0 0, axis 0 0 1, limit lower=0 upper=0.050 effort=400 velocity=0.06
- added joint body_to_chassis: type fixed, parent lift_column, child main_body, origin xyz=0 0 0
- added joint brush_joint: type continuous, parent main_body, child brush, origin xyz=0.20 0 -0.055 rpy=0 1.5708 0, axis 0 0 1
- added joint camera_joint: type fixed, parent main_body, child camera, origin xyz=0.225 0 0.04
- added joint front_bridge_extend1: type prismatic, parent front_bridge_base, child front_bridge_seg1, origin xyz=0.05 0 0, axis 1 0 0, limit lower=0 upper=0.40 effort=250 velocity=0.20
- added joint front_bridge_extend2: type prismatic, parent front_bridge_seg1, child front_bridge_seg2, origin xyz=0.15 0 0, axis 1 0 0, limit lower=0 upper=0.30 effort=200 velocity=0.20
- added joint front_bridge_mount: type fixed, parent main_body, child front_bridge_base, origin xyz=0.18 0 0.010
- added joint front_pad_left_joint: type fixed, parent front_suction_left, child front_pad_left, origin xyz=0 0 -0.032
- added joint front_pad_right_joint: type fixed, parent front_suction_right, child front_pad_right, origin xyz=0 0 -0.032
- added joint front_suction_left_joint: type prismatic, parent front_bridge_seg2, child front_suction_left, origin xyz=0.07 0.07 -0.005, axis 0 0 -1, limit lower=0 upper=0.050 effort=120 velocity=0.08
- added joint front_suction_right_joint: type prismatic, parent front_bridge_seg2, child front_suction_right, origin xyz=0.07 -0.07 -0.005, axis 0 0 -1, limit lower=0 upper=0.050 effort=120 velocity=0.08
- added joint lidar_joint: type fixed, parent main_body, child lidar, origin xyz=0 0 0.08
- added joint rear_bridge_extend1: type prismatic, parent rear_bridge_base, child rear_bridge_seg1, origin xyz=-0.05 0 0, axis -1 0 0, limit lower=0 upper=0.40 effort=250 velocity=0.20
- added joint rear_bridge_extend2: type prismatic, parent rear_bridge_seg1, child rear_bridge_seg2, origin xyz=-0.15 0 0, axis -1 0 0, limit lower=0 upper=0.30 effort=200 velocity=0.20
- added joint rear_bridge_mount: type fixed, parent main_body, child rear_bridge_base, origin xyz=-0.18 0 0.010
- added joint rear_pad_left_joint: type fixed, parent rear_suction_left, child rear_pad_left, origin xyz=0 0 -0.032
- added joint rear_pad_right_joint: type fixed, parent rear_suction_right, child rear_pad_right, origin xyz=0 0 -0.032
- added joint rear_suction_left_joint: type prismatic, parent rear_bridge_seg2, child rear_suction_left, origin xyz=-0.07 0.07 -0.005, axis 0 0 -1, limit lower=0 upper=0.050 effort=120 velocity=0.08
- added joint rear_suction_right_joint: type prismatic, parent rear_bridge_seg2, child rear_suction_right, origin xyz=-0.07 -0.07 -0.005, axis 0 0 -1, limit lower=0 upper=0.050 effort=120 velocity=0.08
- added joint wheel_fl_joint: type continuous, parent main_body, child wheel_fl, origin xyz=0.18 0.175 -0.07 rpy=1.5708 0 0, axis 0 0 1
- added joint wheel_fr_joint: type continuous, parent main_body, child wheel_fr, origin xyz=0.18 -0.175 -0.07 rpy=1.5708 0 0, axis 0 0 1
- added joint wheel_rl_joint: type continuous, parent main_body, child wheel_rl, origin xyz=-0.18 0.175 -0.07 rpy=1.5708 0 0, axis 0 0 1
- added joint wheel_rr_joint: type continuous, parent main_body, child wheel_rr, origin xyz=-0.18 -0.175 -0.07 rpy=1.5708 0 0, axis 0 0 1

Commit message: Changed bridge architecture to gantry-style bridge system

File: solar_robot_pybullet.urdf (robot description, URDF)
Before this commit: robot solar_cleaning_robot, 24 links, 23 joints
Links:
- removed link brush
- removed link camera
- removed link front_bridge_base
- removed link front_bridge_seg1
- removed link front_bridge_seg2
- removed link front_pad_left
- removed link front_pad_right
- removed link front_suction_left
- removed link front_suction_right
- removed link rear_bridge_base
- removed link rear_bridge_seg1
- removed link rear_bridge_seg2
- removed link rear_pad_left
- removed link rear_pad_right
- removed link rear_suction_left
- removed link rear_suction_right
- added link bridge_carriage; visual box size=0.06 0.06 0.06
- added link bridge_link, mass .6; collision box size=1.2 0.08 0.06; visual box size=1.2 0.04 0.04
- added link front_column; visual cylinder length=0.20 radius=0.02
- added link front_left_pad; collision cylinder length=0.01 radius=0.03; visual cylinder length=0.01 radius=0.03
- added link front_plate; visual box size=0.06 0.24 0.02
- added link front_right_pad; collision cylinder length=0.01 radius=0.03; visual cylinder length=0.01 radius=0.03
- added link rear_column; visual cylinder length=0.2 radius=0.02
- added link rear_left_pad; collision cylinder length=0.01 radius=0.03; visual cylinder length=0.01 radius=0.03
- added link rear_plate; visual box size=0.06 0.24 0.02
- added link rear_right_pad; collision cylinder length=0.01 radius=0.03; visual cylinder length=0.01 radius=0.03
- link lidar: geometry visual cylinder length=0.04 radius=0.02
- link lift_column: mass 0.05 -> 0.3; geometry visual cylinder length=0.11 radius=0.02
- link main_body: geometry collision box size=0.35 0.35 0.12; visual box size=0.35 0.35 0.12
Joints:
- removed joint body_lift_joint
- removed joint brush_joint
- removed joint camera_joint
- removed joint front_bridge_extend1
- removed joint front_bridge_extend2
- removed joint front_bridge_mount
- removed joint front_pad_left_joint
- removed joint front_pad_right_joint
- removed joint front_suction_left_joint
- removed joint front_suction_right_joint
- removed joint rear_bridge_extend1
- removed joint rear_bridge_extend2
- removed joint rear_bridge_mount
- removed joint rear_pad_left_joint
- removed joint rear_pad_right_joint
- removed joint rear_suction_left_joint
- removed joint rear_suction_right_joint
- added joint bridge_mount: type prismatic, parent bridge_carriage, child bridge_link, origin xyz=0 0 0, axis 1 0 0, limit lower=-.95 upper=.95 effort=400 velocity=0.4
- added joint column_carriage_joint: type fixed, parent lift_column, child bridge_carriage, origin xyz=0 0 0.085
- added joint front_column_bridge_joint: type fixed, parent bridge_link, child front_column, origin xyz=.58 0 -0.12
- added joint front_left_pad_joint: type fixed, parent front_plate, child front_left_pad, origin xyz=0 0.09 -0.015
- added joint front_plate_column_joint: type fixed, parent front_column, child front_plate, origin xyz=0 0 -0.11
- added joint front_right_pad_joint: type fixed, parent front_plate, child front_right_pad, origin xyz=0 -0.09 -0.015
- added joint lift_column_joint: type prismatic, parent base_link, child lift_column, origin xyz=0 0 0.108, axis 0 0 1, limit lower=-.1 upper=0 effort=500 velocity=0.2
- added joint rear_column_bridge_joint: type fixed, parent bridge_link, child rear_column, origin xyz=-0.58 0 -0.12
- added joint rear_left_pad_joint: type fixed, parent rear_plate, child rear_left_pad, origin xyz=0 0.09 -0.015
- added joint rear_plate_column_joint: type fixed, parent rear_column, child rear_plate, origin xyz=0 0 -0.11
- added joint rear_right_pad_joint: type fixed, parent rear_plate, child rear_right_pad, origin xyz=0 -0.09 -0.015
- joint body_to_chassis: parent lift_column -> base_link
- joint lidar_joint: origin xyz=0 0 0.08 -> xyz=0.198 0 .01 rpy=0 0 1.5708

Commit message: Wheel pos fix. some friction numbers

File: solar_robot_pybullet.urdf (robot description, URDF)
Before this commit: robot solar_cleaning_robot, 18 links, 17 joints
Joints:
- joint wheel_fl_joint: origin xyz=0.18 0.175 -0.07 rpy=1.5708 0 0 -> xyz=0.14 0.175 -0.07 rpy=1.5708 0 0
- joint wheel_fr_joint: origin xyz=0.18 -0.175 -0.07 rpy=1.5708 0 0 -> xyz=0.14 -0.175 -0.07 rpy=1.5708 0 0
- joint wheel_rl_joint: origin xyz=-0.18 0.175 -0.07 rpy=1.5708 0 0 -> xyz=-0.14 0.175 -0.07 rpy=1.5708 0 0
- joint wheel_rr_joint: origin xyz=-0.18 -0.175 -0.07 rpy=1.5708 0 0 -> xyz=-0.14 -0.175 -0.07 rpy=1.5708 0 0

Commit message: marging handling to avoid slipping

File: solar_robot_pybullet.urdf (robot description, URDF)
Before this commit: robot solar_cleaning_robot, 18 links, 17 joints
Joints:
- joint bridge_mount: limit lower=-.93 upper=.93 effort=1000 velocity=0.8 -> lower=-.85 upper=.85 effort=1000 velocity=0.8
